Commit message: debug kdl urdf, debug reset func, init the qpos for arm

File: gymnasium_envs/robot_env_description/ur5e_schunk.urdf (robot description, URDF)
Before this commit: robot ur3, 10 links, 9 joints
Links:
- removed link tool_mid
Joints:
- removed joint wrist_3_link-toolmid_fixed_joint
- joint ee_fixed_joint: origin xyz=0.0 0.092 0.0 rpy=0.0 0.0 1.57079632679 -> xyz=0.0 0.1 0.0 rpy=0.0 0.0 1.5708
- joint elbow_joint: origin xyz=0.0 -0.093 0.244 rpy=0.0 0.0 0.0 -> xyz=0 -0.131 0.425 rpy=0.0 0.0 0.0
- joint shoulder_lift_joint: origin xyz=0.0 0.12 0.0 rpy=0.0 1.570796325 0.0 -> xyz=0.0 0.138 0.0 rpy=0.0 0 0.0
- joint shoulder_pan_joint: origin xyz=0.0 0.0 0.154 rpy=0.0 0.0 3.14 -> xyz=0.0 0.0 0.163 rpy=0.0 0.0 1.5707963
- joint tool_mid-tool0_fixed_joint: origin xyz=-0.142 0.20045 0 rpy=-1.57079632679 0 0 -> xyz=0 0.25 0 rpy=0 0 0; parent tool_mid -> wrist_3_link
- joint wrist_1_joint: origin xyz=0.0 0.0 0.213 rpy=0.0 1.570796325 0.0 -> xyz=0.0 0.0 0.392 rpy=0.0 1.570796325 0.0
- joint wrist_2_joint: origin xyz=0.0 0.104 0.0 rpy=0.0 0.0 0.0 -> xyz=0.0 0.127 0.0 rpy=0.0 0.0 0.0
- joint wrist_3_joint: origin xyz=0.0 0.0 0.08535 rpy=0.0 0.0 0.0 -> xyz=0.0 0.0 0.1 rpy=0.0 0.0 0.0
