Commit message: real trajectory preprocessing

File: gymnasium_envs/robot_env_description/ur5e_schunk_bak.urdf (robot description, URDF)
Before this commit: robot ur5e, 9 links, 8 joints
Joints:
- joint shoulder_lift_joint: origin xyz=0.0 0.138 0.0 rpy=0.0 1.5707963 0.0 -> xyz=0.0 0.138 0.0 rpy=0.0 0 0.0
- joint shoulder_pan_joint: origin xyz=0.0 0.0 0.163 rpy=0.0 0.0 3.1415926 -> xyz=0.0 0.0 0.163 rpy=0.0 0.0 1.5707963
